File: IOB-Adapter-Output_array.brd (EAGLE design)
At the start: 106.7 x 104.1 mm, 133 parts, among them Q1X11 MOSFET-N, Q1X12 MOSFET-N, Q1X21 MOSFET-N, Q1X22 MOSFET-N, Q1X31 MOSFET-N, Q1X32 MOSFET-N, Q1X41 MOSFET-N, Q1X42 MOSFET-N, Q1X51 MOSFET-N, Q1X52 MOSFET-N, Q2X11 MOSFET-N, Q2X12 MOSFET-N, Q2X21 MOSFET-N, Q2X22 MOSFET-N, Q2X31 MOSFET-N, Q2X32 MOSFET-N, Q2X41 MOSFET-N, Q2X42 MOSFET-N, Q2X51 MOSFET-N, Q2X52 MOSFET-N, Q3X11 MOSFET-N, Q3X12 MOSFET-N, Q3X21 MOSFET-N, Q3X22 MOSFET-N, Q3X31 MOSFET-N, Q3X32 MOSFET-N, Q3X41 MOSFET-N, Q3X42 MOSFET-N, Q3X51 MOSFET-N, Q3X52 MOSFET-N, Q4X11 MOSFET-N, Q4X12 MOSFET-N, Q4X21 MOSFET-N, Q4X22 MOSFET-N, Q4X31 MOSFET-N, Q4X32 MOSFET-N, Q4X41 MOSFET-N, Q4X42 MOSFET-N, Q4X51 MOSFET-N, Q4X52 MOSFET-N, Q5X11 MOSFET-N, Q5X12 MOSFET-N, Q5X21 MOSFET-N, Q5X22 MOSFET-N, Q5X31 MOSFET-N, Q5X32 MOSFET-N, Q5X41 MOSFET-N, Q5X42 MOSFET-N, Q5X51 MOSFET-N, Q5X52 MOSFET-N, Q6X11 MOSFET-N, Q6X12 MOSFET-N, Q6X21 MOSFET-N, Q6X22 MOSFET-N, Q6X31 MOSFET-N, Q6X32 MOSFET-N, Q6X41 MOSFET-N, Q6X42 MOSFET-N, Q6X51 MOSFET-N, Q6X52 MOSFET-N, Q7X11 MOSFET-N, Q7X12 MOSFET-N, Q7X21 MOSFET-N, Q7X22 MOSFET-N, Q7X31 MOSFET-N, Q7X32 MOSFET-N, Q7X41 MOSFET-N, Q7X42 MOSFET-N, Q7X51 MOSFET-N, Q7X52 MOSFET-N, Q8X11 MOSFET-N, Q8X12 MOSFET-N, Q8X21 MOSFET-N, Q8X22 MOSFET-N, Q8X31 MOSFET-N, Q8X32 MOSFET-N, Q8X41 MOSFET-N, Q8X42 MOSFET-N, Q8X51 MOSFET-N, Q8X52 MOSFET-N

Commit message: typo in silkscreen
Other:
- board text removed: "Turtle"
Changed lines of the file:
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@@
 <wire x1="25.4" y1="12.7" x2="7.62" y2="12.7" width="0.4064" layer="101"/>
 <wire x1="7.62" y1="12.7" x2="7.62" y2="50.8" width="0.4064" layer="101"/>
-<text x="20.32" y="49.53" size="0.8128" layer="22" font="vector" ratio="10" rot="MR0">Turtle</text>
 <text x="18.415" y="46.355" size="0.762" layer="22" font="vector" ratio="10" rot="MR0">John Plocher</text>
 <text x="24.765" y="47.625" size="0.762" layer="22" font="vector" ratio="10" rot="MR0">2020.09</text>
@@
 <wire x1="25.4" y1="50.8" x2="7.62" y2="50.8" width="0.4064" layer="101"/>
 <wire x1="7.62" y1="50.8" x2="7.62" y2="88.9" width="0.4064" layer="101"/>
-<text x="20.32" y="87.63" size="0.8128" layer="22" font="vector" ratio="10" rot="MR0">Turtle</text>
+<text x="24.13" y="86.995" size="0.8128" layer="22" font="vector" ratio="10" rot="MR0">Open Drain Output</text>
 <text x="18.415" y="84.455" size="0.762" layer="22" font="vector" ratio="10" rot="MR0">John Plocher</text>
 <text x="24.765" y="85.725" size="0.762" layer="22" font="vector" ratio="10" rot="MR0">2020.09</text>
@@
 <wire x1="43.18" y1="12.7" x2="25.4" y2="12.7" width="0.4064" layer="101"/>
 <wire x1="25.4" y1="12.7" x2="25.4" y2="50.8" width="0.4064" layer="101"/>
-<text x="38.1" y="49.53" size="0.8128" layer="22" font="vector" ratio="10" rot="MR0">Turtle</text>
 <text x="36.195" y="46.355" size="0.762" layer="22" font="vector" ratio="10" rot="MR0">John Plocher</text>
 <text x="42.545" y="47.625" size="0.762" layer="22" font="vector" ratio="10" rot="MR0">2020.09</text>
@@
 <wire x1="43.18" y1="50.8" x2="25.4" y2="50.8" width="0.4064" layer="101"/>
 <wire x1="25.4" y1="50.8" x2="25.4" y2="88.9" width="0.4064" layer="101"/>
-<text x="38.1" y="87.63" size="0.8128" layer="22" font="vector" ratio="10" rot="MR0">Turtle</text>
 <text x="36.195" y="84.455" size="0.762" layer="22" font="vector" ratio="10" rot="MR0">John Plocher</text>
 <text x="42.545" y="85.725" size="0.762" layer="22" font="vector" ratio="10" rot="MR0">2020.09</text>
@@
 <wire x1="60.96" y1="12.7" x2="43.18" y2="12.7" width="0.4064" layer="101"/>
 <wire x1="43.18" y1="12.7" x2="43.18" y2="50.8" width="0.4064" layer="101"/>
-<text x="55.88" y="49.53" size="0.8128" layer="22" font="vector" ratio="10" rot="MR0">Turtle</text>
 <text x="53.975" y="46.355" size="0.762" layer="22" font="vector" ratio="10" rot="MR0">John Plocher</text>
 <text x="60.325" y="47.625" size="0.762" layer="22" font="vector" ratio="10" rot="MR0">2020.09</text>
@@
 <wire x1="60.96" y1="50.8" x2="43.18" y2="50.8" width="0.4064" layer="101"/>
 <wire x1="43.18" y1="50.8" x2="43.18" y2="88.9" width="0.4064" layer="101"/>
-<text x="55.88" y="87.63" size="0.8128" layer="22" font="vector" ratio="10" rot="MR0">Turtle</text>
 <text x="53.975" y="84.455" size="0.762" layer="22" font="vector" ratio="10" rot="MR0">John Plocher</text>
 <text x="60.325" y="85.725" size="0.762" layer="22" font="vector" ratio="10" rot="MR0">2020.09</text>
@@
 <wire x1="78.74" y1="12.7" x2="60.96" y2="12.7" width="0.4064" layer="101"/>
 <wire x1="60.96" y1="12.7" x2="60.96" y2="50.8" width="0.4064" layer="101"/>
-<text x="73.66" y="49.53" size="0.8128" layer="22" font="vector" ratio="10" rot="MR0">Turtle</text>
 <text x="71.755" y="46.355" size="0.762" layer="22" font="vector" ratio="10" rot="MR0">John Plocher</text>
 <text x="78.105" y="47.625" size="0.762" layer="22" font="vector" ratio="10" rot="MR0">2020.09</text>
@@
 <wire x1="78.74" y1="50.8" x2="60.96" y2="50.8" width="0.4064" layer="101"/>
 <wire x1="60.96" y1="50.8" x2="60.96" y2="88.9" width="0.4064" layer="101"/>
-<text x="73.66" y="87.63" size="0.8128" layer="22" font="vector" ratio="10" rot="MR0">Turtle</text>
 <text x="71.755" y="84.455" size="0.762" layer="22" font="vector" ratio="10" rot="MR0">John Plocher</text>
 <text x="78.105" y="85.725" size="0.762" layer="22" font="vector" ratio="10" rot="MR0">2020.09</text>
@@
 <wire x1="96.52" y1="12.7" x2="78.74" y2="12.7" width="0.4064" layer="101"/>
 <wire x1="78.74" y1="12.7" x2="78.74" y2="50.8" width="0.4064" layer="101"/>
-<text x="91.44" y="49.53" size="0.8128" layer="22" font="vector" ratio="10" rot="MR0">Turtle</text>
 <text x="89.535" y="46.355" size="0.762" layer="22" font="vector" ratio="10" rot="MR0">John Plocher</text>
 <text x="95.885" y="47.625" size="0.762" layer="22" font="vector" ratio="10" rot="MR0">2020.09</text>
@@
 <wire x1="96.52" y1="50.8" x2="78.74" y2="50.8" width="0.4064" layer="101"/>
 <wire x1="78.74" y1="50.8" x2="78.74" y2="88.9" width="0.4064" layer="101"/>
-<text x="91.44" y="87.63" size="0.8128" layer="22" font="vector" ratio="10" rot="MR0">Turtle</text>
 <text x="89.535" y="84.455" size="0.762" layer="22" font="vector" ratio="10" rot="MR0">John Plocher</text>
 <text x="95.885" y="85.725" size="0.762" layer="22" font="vector" ratio="10" rot="MR0">2020.09</text>
@@
 <text x="34.925" y="93.98" size="3.81" layer="21" font="vector" ratio="10">Open Drain Output</text>
 <text x="82.55" y="91.44" size="1.778" layer="21" font="vector" ratio="10">v1.0</text>
+<text x="41.91" y="86.995" size="0.8128" layer="22" font="vector" ratio="10" rot="MR0">Open Drain Output</text>
+<text x="59.69" y="86.995" size="0.8128" layer="22" font="vector" ratio="10" rot="MR0">Open Drain Output</text>
+<text x="77.47" y="86.995" size="0.8128" layer="22" font="vector" ratio="10" rot="MR0">Open Drain Output</text>
+<text x="95.25" y="86.995" size="0.8128" layer="22" font="vector" ratio="10" rot="MR0">Open Drain Output</text>
+<text x="24.13" y="48.895" size="0.8128" layer="22" font="vector" ratio="10" rot="MR0">Open Drain Output</text>
+<text x="41.91" y="48.895" size="0.8128" layer="22" font="vector" ratio="10" rot="MR0">Open Drain Output</text>
+<text x="59.69" y="48.895" size="0.8128" layer="22" font="vector" ratio="10" rot="MR0">Open Drain Output</text>
+<text x="77.47" y="48.895" size="0.8128" layer="22" font="vector" ratio="10" rot="MR0">Open Drain Output</text>
+<text x="95.25" y="48.895" size="0.8128" layer="22" font="vector" ratio="10" rot="MR0">Open Drain Output</text>
 </plain>
 <attributes>

Commit message: added values for connectors
Parts:
- CARRIER: value (none) -> 10x10
- FID-LR, FID-UL: value (none) -> FIDUCIAL
Changed lines of the file:
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@@
 <element name="R3X52" library="SPCoast" package="0805-RES" value="10k" x="89.916" y="68.453" rot="R90"/>
 <element name="R4X52" library="SPCoast" package="0805-RES" value="10k" x="93.726" y="68.453" rot="R90"/>
-<element name="CARRIER" library="SPCoast" package="BOARD-DINRAIL-3.17IN-5X2-IOP" value="" x="0" y="0"/>
-<element name="FID-UL" library="SPCoast" package="FIDUCIAL_1MM" value="" x="5.08" y="91.44" smashed="yes">
+<element name="CARRIER" library="SPCoast" package="BOARD-DINRAIL-3.17IN-5X2-IOP" value="10x10" x="0" y="0"/>
+<element name="FID-UL" library="SPCoast" package="FIDUCIAL_1MM" value="FIDUCIAL" x="5.08" y="91.44" smashed="yes">
 <attribute name="NAME" x="2.54" y="89.535" size="1.016" layer="25" rot="R90"/>
 </element>
-<element name="FID-LR" library="SPCoast" package="FIDUCIAL_1MM" value="" x="93.98" y="10.16" smashed="yes">
+<element name="FID-LR" library="SPCoast" package="FIDUCIAL_1MM" value="FIDUCIAL" x="93.98" y="10.16" smashed="yes">
 <attribute name="NAME" x="99.06" y="6.985" size="1.016" layer="25" rot="R90"/>
 </element>

Commit message: normalized values
Parts:
- CARRIER: value 10x10 -> BOARD
- Q1X11, Q1X12, Q1X21, Q1X22, Q1X31, Q1X32, Q1X41, Q1X42, Q1X51, Q1X52, Q2X11, Q2X12, Q2X21, Q2X22, Q2X31, Q2X32, Q2X41, Q2X42, Q2X51, Q2X52, Q3X11, Q3X12, Q3X21, Q3X22, Q3X31, Q3X32, Q3X41, Q3X42, Q3X51, Q3X52, Q4X11, Q4X12, Q4X21, Q4X22, Q4X31, Q4X32, Q4X41, Q4X42, Q4X51, Q4X52, Q5X11, Q5X12, Q5X21, Q5X22, Q5X31, Q5X32, Q5X41, Q5X42, Q5X51, Q5X52, Q6X11, Q6X12, Q6X21, Q6X22, Q6X31, Q6X32, Q6X41, Q6X42, Q6X51, Q6X52, Q7X11, Q7X12, Q7X21, Q7X22, Q7X31, Q7X32, Q7X41, Q7X42, Q7X51, Q7X52, Q8X11, Q8X12, Q8X21, Q8X22, Q8X31, Q8X32, Q8X41, Q8X42, Q8X51, Q8X52: value MOSFET-N -> N-FET
